File: PCB_Stop_BBM_3PIC_Prog/Stop_BBM_3PIC.sch (KiCad schematic (older format))
At the start: 6 parts, among them J1 Haut parleur (MOUSE), J2 Conn_01x05_Male, J3 Conn_01x06, J4 Conn_01x01_Male, J5 Conn_01x01_Male, J6 Conn_01x01_Male

Commit message: Modifié pour EUROCIRCUIT  + Devis
discuter de la sérigraphie
Other:
- note added: "BED OF NAILS STOP_BSB_3PIC"
- note added: "ICSP Programming connector"
- note added: "ICSP Programming with probes"
- note added: "ICSPDAT probes for PIC10 and PIC12"
- note added: "Probes for mechanical support"
- note added: "pick signal on HP"
- note removed: "ICSP Programming"
- moved on the sheet: J1, J4, J5, J6
Changed lines of the file:
@@
 EESchema Schematic File Version 4
+LIBS:Stop_BBM_3PIC-cache
 EELAYER 30 0
 EELAYER END
@@
 encoding utf-8
 Sheet 1 1
-Title "Stop_BSB_3PIC"
+Title "Bed of Nails Stop_BSB_3PIC"
 Date "2022-02-03"
-Rev "V1.1"
+Rev "for V1.1"
 Comp "ADTP"
 Comment1 "Voir Readme.txt"
 Comment2 "https://github.com/benoitGIRAUD/STOP_BBM_3PIC"
-Comment3 ""
+Comment3 "Auteur: Benoît"
 Comment4 ""
 $EndDescr
@@
 	4915 5050 4915 7600
 Text Notes 4905 5030 0    50   ~ 0
-ICSP Programming
+ICSP Programming with probes
 Wire Wire Line
 	5890 6660 5890 7295
@@
 L Stop_BBM_3PIC-rescue:Conn_01x02_Male-connecteur-dagostino_stop_BirdBuzzMouse-rescue J1
 U 1 1 6064EA3D
-P 4750 4450
-F 0 "J1" V 4904 4262 50  0000 R CNN
-F 1 "Haut parleur (MOUSE)" V 4813 4262 50  0000 R CNN
-F 2 "Stop_BBM_3PIC:SolderWirePad_1x01_SMD_5x10mm_BBM" H 4750 4450 50  0001 C CNN
-F 3 "https://www.farnell.com/datasheets/2861450.pdf" H 4750 4450 50  0001 C CNN
-F 4 "PRO SIGNAL" V 4750 4450 50  0001 C CNN "Manufacturer"
-F 5 "ABS-209-RC" V 4750 4450 50  0001 C CNN "Manufacturer PN"
-F 6 "" V 4750 4450 50  0001 C CNN "DNP"
-F 7 "A0020419" V 4750 4450 50  0001 C CNN "Code_X3"
-F 8 "Haut-parleur, Mini, Cone Mylar, 0.25 W, 32 ohms, 500 Hz à 5500 Hz" V 4750 4450 50  0001 C CNN "DESIGNATION"
-	1    4750 4450
+P 5270 4210
+F 0 "J1" V 5424 4022 50  0000 R CNN
+F 1 "Haut parleur (MOUSE)" V 5333 4022 50  0000 R CNN
+F 2 "Stop_BBM_3PIC:SolderWirePad_1x01_SMD_5x10mm_BBM" H 5270 4210 50  0001 C CNN
+F 3 "https://www.farnell.com/datasheets/2861450.pdf" H 5270 4210 50  0001 C CNN
+F 4 "PRO SIGNAL" V 5270 4210 50  0001 C CNN "Manufacturer"
+F 5 "ABS-209-RC" V 5270 4210 50  0001 C CNN "Manufacturer PN"
+F 6 "" V 5270 4210 50  0001 C CNN "DNP"
+F 7 "A0020419" V 5270 4210 50  0001 C CNN "Code_X3"
+F 8 "Haut-parleur, Mini, Cone Mylar, 0.25 W, 32 ohms, 500 Hz à 5500 Hz" V 5270 4210 50  0001 C CNN "DESIGNATION"
+	1    5270 4210
 	0    -1   -1   0
 $EndComp
@@
 Wire Wire Line
 	9000 6000 8700 6000
-NoConn ~ 4750 4250
-Text GLabel 4850 3850 1    50   BiDi ~ 0
+NoConn ~ 5270 4010
+Text GLabel 5370 3610 1    50   BiDi ~ 0
 ISCPDAT
 $Comp
 L Connector:Conn_01x01_Male J4
 U 1 1 62B4C517
-P 5200 4000
-F 0 "J4" H 5172 3932 50  0000 R CNN
-F 1 "Conn_01x01_Male" H 5172 4023 50  0000 R CNN
-F 2 "PinHeader_1x01_P2.54mm_Vertical" H 5200 4000 50  0001 C CNN
-F 3 "~" H 5200 4000 50  0001 C CNN
-	1    5200 4000
+P 5720 3760
+F 0 "J4" H 5692 3692 50  0000 R CNN
+F 1 "Conn_01x01_Male" H 5692 3783 50  0000 R CNN
+F 2 "PinHeader_1x01_P2.54mm_Vertical" H 5720 3760 50  0001 C CNN
+F 3 "~" H 5720 3760 50  0001 C CNN
+	1    5720 3760
 	-1   0    0    1
 $EndComp
 Wire Wire Line
-	4850 3850 4850 4000
-Wire Wire Line
-	5000 4000 4850 4000
-Connection ~ 4850 4000
-Wire Wire Line
-	4850 4000 4850 4250
+	5370 3610 5370 3760
+Wire Wire Line
+	5520 3760 5370 3760
+Connection ~ 5370 3760
+Wire Wire Line
+	5370 3760 5370 4010
 $Comp
 L Connector:Conn_01x01_Male J6
 U 1 1 62B4D8D0
-P 6700 4000
-F 0 "J6" H 6672 3932 50  0000 R CNN
-F 1 "Conn_01x01_Male" H 6672 4023 50  0000 R CNN
-F 2 "PinHeader_1x01_P2.54mm_Vertical" H 6700 4000 50  0001 C CNN
-F 3 "~" H 6700 4000 50  0001 C CNN
-	1    6700 4000
+P 8640 4070
+F 0 "J6" H 8612 4002 50  0000 R CNN
+F 1 "Conn_01x01_Male" H 8612 4093 50  0000 R CNN
+F 2 "PinHeader_1x01_P2.54mm_Vertical" H 8640 4070 50  0001 C CNN
+F 3 "~" H 8640 4070 50  0001 C CNN
+	1    8640 4070
 	-1   0    0    1
 $EndComp
@@
 L Connector:Conn_01x01_Male J5
 U 1 1 62B4E1F8
-P 6700 3500
-F 0 "J5" H 6672 3432 50  0000 R CNN
-F 1 "Conn_01x01_Male" H 6672 3523 50  0000 R CNN
-F 2 "PinHeader_1x01_P2.54mm_Vertical" H 6700 3500 50  0001 C CNN
-F 3 "~" H 6700 3500 50  0001 C CNN
-	1    6700 3500
+P 8640 3570
+F 0 "J5" H 8612 3502 50  0000 R CNN
+F 1 "Conn_01x01_Male" H 8612 3593 50  0000 R CNN
+F 2 "PinHeader_1x01_P2.54mm_Vertical" H 8640 3570 50  0001 C CNN
+F 3 "~" H 8640 3570 50  0001 C CNN
+	1    8640 3570
 	-1   0    0    1
 $EndComp
-NoConn ~ 6500 4000
-NoConn ~ 6500 3500
+NoConn ~ 8440 4070
+NoConn ~ 8440 3570
+Text Notes 3430 1460 0    236  Italic 47
+BED OF NAILS STOP_BSB_3PIC
+Wire Notes Line
+	8000 5050 10050 5050
+Wire Notes Line
+	10050 5050 10050 6420
+Wire Notes Line
+	10050 6420 8000 6420
+Wire Notes Line
+	8000 5050 8000 6420
+Text Notes 8000 5000 0    50   ~ 0
+ICSP Programming connector
+Wire Notes Line
+	4920 3080 6910 3080
+Wire Notes Line
+	6910 3080 6910 4670
+Wire Notes Line
+	6910 4670 4920 4670
+Wire Notes Line
+	4920 3080 4920 4670
+Wire Notes Line
+	8010 4670 8010 3080
+Wire Notes Line
+	8010 3080 10050 3080
+Wire Notes Line
+	10050 3080 10050 4670
+Wire Notes Line
+	10050 4670 8010 4670
+Text Notes 4905 3040 0    50   ~ 0
+ICSPDAT probes for PIC10 and PIC12
+Text Notes 8010 3040 0    50   ~ 0
+Probes for mechanical support
+Text Notes 5370 4420 0    50   ~ 0
+pick signal on HP
 $EndSCHEMATC

Commit message: PRODUCTION: Démo semaine prochaine
Other:
- note added: "0.8 mm de diamètre pour rentrer en force le fût"
Changed lines of the file:
@@
 EESchema Schematic File Version 4
-LIBS:Stop_BBM_3PIC-cache
 EELAYER 30 0
 EELAYER END
@@
 Text Notes 5370 4420 0    50   ~ 0
 pick signal on HP
+Text Notes 4915 7715 0    50   ~ 0
+0.8 mm de diamètre pour rentrer en force le fût
 $EndSCHEMATC
